File: micromouse/untitled.kicad_sch (KiCad schematic)
At the start: 15 parts, among them IC1 STM32F205RET7, SW1 CK_KMS2xxG

Commit message: updated footprints and schematic
Parts:
- C11, C71, C72, C74, C76, C77, C9: footprint CL21B104KBCNNNC:CAPC2012X95N -> Capacitor_SMD:C_0805_2012Metric
- C25: footprint CL21B106KOQNNNE:CAPC2012X140N -> Capacitor_SMD:C_0805_2012Metric
- C70: footprint GRM21BR71C105KA01L:CAPC2012X135N -> Capacitor_SMD:C_0805_2012Metric
- C73, C75: footprint GRM21BR71A225KA01L:CAPC2012X135N -> Capacitor_SMD:C_0805_2012Metric
- IC1: footprint QFP50P1200X1200X160-64N -> STM32F205RET7:QFP50P1200X1200X160-64N
- R5, R6: footprint WK73R2ATTD103J:RESC1220X65N -> Resistor_SMD:R_0805_2012Metric
Changed lines of the file:
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@@
 			)
 		)
-		(property "Footprint" "GRM21BR71C105KA01L:CAPC2012X135N"
+		(property "Footprint" "Capacitor_SMD:C_0805_2012Metric"
 			(at 55.88 110.49 0)
 			(effects
@@
 			)
 		)
-		(property "Footprint" "QFP50P1200X1200X160-64N"
+		(property "Footprint" "STM32F205RET7:QFP50P1200X1200X160-64N"
 			(at 128.27 159.69 0)
 			(effects
@@
 		)
 		(instances
-			(project "micromouse"
+			(project ""
+				(path "/6f21d099-3493-45a5-8fb2-59b651d74bbe"
+					(reference "IC1")
+					(unit 1)
+				)
 				(path "/6f21d099-3493-45a5-8fb2-59b651d74bbe/0e2a7964-9a2d-4139-b18d-934c264bbaa5"
 					(reference "IC1")
@@
 			)
 		)
-		(property "Footprint" "GRM21BR71A225KA01L:CAPC2012X135N"
+		(property "Footprint" "Capacitor_SMD:C_0805_2012Metric"
 			(at 121.92 139.7 0)
 			(effects
@@
 			)
 		)
-		(property "Footprint" "CL21B104KBCNNNC:CAPC2012X95N"
+		(property "Footprint" "Capacitor_SMD:C_0805_2012Metric"
 			(at 77.47 72.39 0)
 			(effects
@@
 			)
 		)
-		(property "Footprint" "WK73R2ATTD103J:RESC1220X65N"
+		(property "Footprint" "Resistor_SMD:R_0805_2012Metric"
 			(at 114.3 146.05 0)
 			(effects
@@
 			)
 		)
-		(property "Footprint" "CL21B104KBCNNNC:CAPC2012X95N"
+		(property "Footprint" "Capacitor_SMD:C_0805_2012Metric"
 			(at 68.58 107.95 0)
 			(effects
@@
 			)
 		)
-		(property "Footprint" "CL21B104KBCNNNC:CAPC2012X95N"
+		(property "Footprint" "Capacitor_SMD:C_0805_2012Metric"
 			(at 81.28 46.99 0)
 			(effects
@@
 			)
 		)
-		(property "Footprint" "CL21B104KBCNNNC:CAPC2012X95N"
+		(property "Footprint" "Capacitor_SMD:C_0805_2012Metric"
 			(at 154.94 72.39 0)
 			(effects
@@
 			)
 		)
-		(property "Footprint" "CL21B104KBCNNNC:CAPC2012X95N"
+		(property "Footprint" "Capacitor_SMD:C_0805_2012Metric"
 			(at 95.25 140.97 0)
 			(effects
@@
 			)
 		)
-		(property "Footprint" "CL21B106KOQNNNE:CAPC2012X140N"
+		(property "Footprint" "Capacitor_SMD:C_0805_2012Metric"
 			(at 95.25 151.13 0)
 			(effects
@@
 			)
 		)
-		(property "Footprint" "GRM21BR71A225KA01L:CAPC2012X135N"
+		(property "Footprint" "Capacitor_SMD:C_0805_2012Metric"
 			(at 137.16 77.47 0)
 			(effects
@@
 			)
 		)
-		(property "Footprint" "WK73R2ATTD103J:RESC1220X65N"
+		(property "Footprint" "Resistor_SMD:R_0805_2012Metric"
 			(at 96.52 43.18 0)
 			(effects
@@
 			)
 		)
-		(property "Footprint" "CL21B104KBCNNNC:CAPC2012X95N"
+		(property "Footprint" "Capacitor_SMD:C_0805_2012Metric"
 			(at 127 154.94 0)
 			(effects
@@
 			)
 		)
-		(property "Footprint" "CL21B104KBCNNNC:CAPC2012X95N"
+		(property "Footprint" "Capacitor_SMD:C_0805_2012Metric"
 			(at 213.36 71.12 0)
 			(effects

Commit message: updates to layout
Connections:
- net PC5: now reaches IC1.25 (PC5)
- net I2C1_SCL renamed SCL
- net I2C1_SDA renamed SDA
- no-connect marks 0 -> 47
Changed lines of the file:
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@@
 		(color 0 0 0 0)
 	)
+	(no_connect
+		(at 99.06 130.81)
+	)
+	(no_connect
+		(at 78.74 97.79)
+	)
+	(no_connect
+		(at 132.08 82.55)
+	)
+	(no_connect
+		(at 78.74 80.01)
+	)
+	(no_connect
+		(at 101.6 130.81)
+	)
+	(no_connect
+		(at 111.76 130.81)
+	)
+	(no_connect
+		(at 114.3 57.15)
+	)
+	(no_connect
+		(at 78.74 82.55)
+	)
+	(no_connect
+		(at 116.84 57.15)
+	)
+	(no_connect
+		(at 78.74 92.71)
+	)
+	(no_connect
+		(at 104.14 130.81)
+	)
+	(no_connect
+		(at 93.98 57.15)
+	)
+	(no_connect
+		(at 78.74 100.33)
+	)
+	(no_connect
+		(at 109.22 57.15)
+	)
+	(no_connect
+		(at 132.08 102.87)
+	)
+	(no_connect
+		(at 78.74 95.25)
+	)
+	(no_connect
+		(at 78.74 113.03)
+	)
+	(no_connect
+		(at 109.22 130.81)
+	)
+	(no_connect
+		(at 132.08 90.17)
+	)
+	(no_connect
+		(at 132.08 113.03)
+	)
+	(no_connect
+		(at 119.38 57.15)
+	)
+	(no_connect
+		(at 104.14 57.15)
+	)
+	(no_connect
+		(at 78.74 77.47)
+	)
+	(no_connect
+		(at 132.08 85.09)
+	)
+	(no_connect
+		(at 96.52 130.81)
+	)
+	(no_connect
+		(at 132.08 100.33)
+	)
+	(no_connect
+		(at 116.84 130.81)
+	)
+	(no_connect
+		(at 132.08 110.49)
+	)
+	(no_connect
+		(at 91.44 57.15)
+	)
+	(no_connect
+		(at 106.68 57.15)
+	)
+	(no_connect
+		(at 111.76 57.15)
+	)
+	(no_connect
+		(at 132.08 92.71)
+	)
+	(no_connect
+		(at 78.74 107.95)
+	)
+	(no_connect
+		(at 93.98 130.81)
+	)
+	(no_connect
+		(at 86.36 130.81)
+	)
+	(no_connect
+		(at 132.08 105.41)
+	)
+	(no_connect
+		(at 132.08 97.79)
+	)
+	(no_connect
+		(at 78.74 87.63)
+	)
+	(no_connect
+		(at 121.92 57.15)
+	)
+	(no_connect
+		(at 88.9 57.15)
+	)
+	(no_connect
+		(at 119.38 130.81)
+	)
+	(no_connect
+		(at 132.08 107.95)
+	)
+	(no_connect
+		(at 132.08 95.25)
+	)
+	(no_connect
+		(at 124.46 57.15)
+	)
+	(no_connect
+		(at 78.74 110.49)
+	)
+	(no_connect
+		(at 78.74 85.09)
+	)
+	(no_connect
+		(at 132.08 87.63)
+	)
 	(wire
 		(pts
@@
 		)
 	)
+	(global_label "SCL"
+		(shape input)
+		(at 101.6 52.07 90)
+		(fields_autoplaced yes)
+		(effects
+			(font
+				(size 1.27 1.27)
+			)
+			(justify left)
+		)
+		(property "Intersheetrefs" "${INTERSHEET_REFS}"
+			(at 101.6 45.5772 90)
+			(effects
+				(font
+					(size 1.27 1.27)
+				)
+				(justify left)
+				(hide yes)
+			)
+		)
+	)
 	(global_label "GND"
 		(shape input)
@@
 		)
 	)
+	(global_label "SDA"
+		(shape input)
+		(at 99.06 52.07 90)
+		(fields_autoplaced yes)
+		(effects
+			(font
+				(size 1.27 1.27)
+			)
+			(justify left)
+		)
+		(property "Intersheetrefs" "${INTERSHEET_REFS}"
+			(at 99.06 45.5167 90)
+			(effects
+				(font
+					(size 1.27 1.27)
+				)
+				(justify left)
+				(hide yes)
+			)
+		)
+	)
 	(global_label "GND"
 		(shape input)
@@
 		)
 	)
-	(global_label "I2C1_SDA"
-		(shape input)
-		(at 99.06 52.07 90)
-		(fields_autoplaced yes)
-		(effects
-			(font
-				(size 1.27 1.27)
-			)
-			(justify left)
-		)
-		(property "Intersheetrefs" "${INTERSHEET_REFS}"
-			(at 99.06 40.2553 90)
-			(effects
-				(font
-					(size 1.27 1.27)
-				)
-				(justify left)
-				(hide yes)
-			)
-		)
-	)
 	(global_label "GND"
 		(shape input)
@@
 		)
 	)
-	(global_label "I2C1_SCL"
-		(shape input)
-		(at 101.6 52.07 90)
-		(fields_autoplaced yes)
-		(effects
-			(font
-				(size 1.27 1.27)
-			)
-			(justify left)
-		)
-		(property "Intersheetrefs" "${INTERSHEET_REFS}"
-			(at 101.6 40.3158 90)
-			(effects
-				(font
-					(size 1.27 1.27)
-				)
-				(justify left)
-				(hide yes)
-			)
-		)
-	)
 	(global_label "3V3"
 		(shape input)
@@
 			(effects
 				(font
+					(size 1.27 1.27)
+				)
+				(justify right)
+				(hide yes)
+			)
+		)
+	)
+	(global_label "PC5"
+		(shape input)
+		(at 106.68 130.81 270)
+		(fields_autoplaced yes)
+		(effects
+			(font
+				(size 1.27 1.27)
+			)
+			(justify right)
+		)
+		(property "Intersheetrefs" "${INTERSHEET_REFS}"
+			(at 106.68 137.5447 90)
+			(effects
+				(font
