File: micromouse/ir-emitter-receiver.kicad_sch (KiCad schematic)
At the start: 48 parts, among them Q1 SFH_313_FA-3_4, Q2 SFH_313_FA-3_4, Q3 SFH_313_FA-3_4, Q4 SFH_313_FA-3_4, U1 BS170, U4 BS170, U6 BS170, U7 BS170

Commit message: pcb updates
Parts:
- removed U1, U4, U6, U7: BS170, bs170:TO_SA06_ONS, symbol nchannelmosfet-mm:BS170
- added Q5, Q6, Q7, Q8: 2N7002LT1G, new_n_channel_mosfets:SOT95P240X111-3N, symbol new_n_channel_mosfet:2N7002LT1G
Connections:
- net GND: now also Q5.2, Q6.2, Q7.2, Q8.2
- net at R1.1, R3.2: now also Q5.1
- net at LED1.1: now also Q5.3
- net at R19.2, R20.1: now also Q7.1
- net at LED11.1: now also Q7.3
- net at LED5.1: now also Q6.3
- net at R10.1, R9.2: now also Q6.1
- net at R14.2, R15.1: now also Q8.1
- net at LED8.1: now also Q8.3
- net PA5 renamed PC6
- net PA6 renamed PC0
