File: micromouse/mcu.kicad_sch (KiCad schematic)
At the start: 15 parts

Commit message: updates to layout
Parts:
- removed C1, C3, C4: 0.1 uF, CL21B104KBCNNNC:CAPC2012X95N, symbol CL21B104KBCNNNC:CL21B104KBCNNNC
- removed C2: 1 uF, GRM21BR71C105KA01L:CAPC2012X135N, symbol GRM21BR71C105KA01L:GRM21BR71C105KA01L
- removed C5: 10 uF, CL21B106KOQNNNE:CAPC2012X140N, symbol CL21B106KOQNNNE:CL21B106KOQNNNE
- removed C6: 2.2uF, GRM21BR71A225KA01L:CAPC2012X135N, symbol GRM21BR71A225KA01L:GRM21BR71A225KA01L
- removed R1, R2: 10k, WK73R2ATTD103J:RESC1220X65N, symbol WK73R2ATTD103J:WK73R2ATTD103J
- added C25: 10 uF, Capacitor_SMD:C_0805_2012Metric, symbol CL21B106KOQNNNE:CL21B106KOQNNNE
- added C70: 1 uF, Capacitor_SMD:C_0805_2012Metric, symbol GRM21BR71C105KA01L:GRM21BR71C105KA01L
- added C71, C72, C9: 0.1 uF, Capacitor_SMD:C_0805_2012Metric, symbol CL21B104KBCNNNC:CL21B104KBCNNNC
- added C73: 2.2uF, Capacitor_SMD:C_0805_2012Metric, symbol GRM21BR71A225KA01L:GRM21BR71A225KA01L
- added R5, R6: 10k, Resistor_SMD:R_0805_2012Metric, symbol WK73R2ATTD103J:WK73R2ATTD103J
- C11: footprint CL21B104KBCNNNC:CAPC2012X95N -> Capacitor_SMD:C_0805_2012Metric
- C74: renamed from C7; footprint CL21B104KBCNNNC:CAPC2012X95N -> Capacitor_SMD:C_0805_2012Metric
- C75: renamed from C8; footprint GRM21BR71A225KA01L:CAPC2012X135N -> Capacitor_SMD:C_0805_2012Metric
- C76: renamed from C9; footprint CL21B104KBCNNNC:CAPC2012X95N -> Capacitor_SMD:C_0805_2012Metric
- C77: renamed from C10; footprint CL21B104KBCNNNC:CAPC2012X95N -> Capacitor_SMD:C_0805_2012Metric
- IC1: renamed from IC?; footprint QFP50P1200X1200X160-64N -> STM32F205RET7:QFP50P1200X1200X160-64N
- gave numbers to parts that had none: 1
Connections:
- net 3V3: now also C25.1, C70.1, C71.1, C72.1, C9.1
- net GND: now also SW1.SH (B), C25.2, C70.2, C71.2, C72.2, C73.2, C9.2, R5.1, R6.1
- net at IC1.60 (BOOT0): now also R5.2
- net at IC1.28 (PB2): now also R6.2
- net PC2: now reaches IC1.10 (PC2)
- net PA1: now reaches IC1.15 (PA1)
- net PA2: now reaches IC1.16 (PA2)
- net PA4: now reaches IC1.20 (PA4)
- net PA5: now reaches IC1.21 (PA5)
- net PC5: now reaches IC1.25 (PC5)
- net at IC1.31 (VCAP_1): now also C73.1
- net PC1: now reaches IC1.9 (PC1)
- net I2C1_SCL renamed SCL
- net I2C1_SDA renamed SDA
- no-connect marks 0 -> 41
Other:
- moved on the sheet: C74, C75, C76, C77, IC1, SW1

Commit message: pcb updates
Parts:
- added J5: Conn_01x04_Pin, Connector_PinHeader_2.54mm:PinHeader_1x04_P2.54mm_Vertical, symbol Connector:Conn_01x04_Pin
Connections:
- net 3V3: now also J5.4 (Pin_4)
- net GND: now also J5.2 (Pin_2)
- net SWCLK: now also J5.1 (Pin_1)
- net SWDIO: now also J5.3 (Pin_3)
- net PA3: now reaches IC1.17 (PA3)
- net PA6: now reaches IC1.22 (PA6)
- net PA7: now reaches IC1.23 (PA7)
- net PC6: now reaches IC1.37 (PC6)
- net PC9: now reaches IC1.40 (PC9)
- net LENC2: now reaches IC1.41 (PA8)
- net LENC1: now reaches IC1.42 (PA9)
- net RENC2: now reaches IC1.56 (PB4)
- net RENC1: now reaches IC1.57 (PB5)
- net PB9: now reaches IC1.62 (PB9)
- net PC0: now reaches IC1.8 (PC0)
- no-connect marks 41 -> 30
Other:
- note added: "Debug Pin Headers"
