File: micromouse - KiCAD Files/mcu.kicad_sch (KiCad schematic)
At the start: 15 parts, among them IC1 STM32F205RET7, SW1 CK_KMS2xxG

Commit message: file management
Parts:
- added J5: Conn_01x04_Pin, Connector_PinHeader_2.54mm:PinHeader_1x04_P2.54mm_Vertical, symbol Connector:Conn_01x04_Pin
Connections:
- net 3V3: now also J5.4 (Pin_4)
- net GND: now also SW1.SH (B), J5.2 (Pin_2)
- net SWCLK: now also J5.1 (Pin_1)
- net SWDIO: now also J5.3 (Pin_3)
- net PC2: now reaches IC1.10 (PC2)
- net PA1: now reaches IC1.15 (PA1)
- net PA2: now reaches IC1.16 (PA2)
- net PA3: now reaches IC1.17 (PA3)
- net PA4: now reaches IC1.20 (PA4)
- net PA5: now reaches IC1.21 (PA5)
- net PA6: now reaches IC1.22 (PA6)
- net PA7: now reaches IC1.23 (PA7)
- net PC6: now reaches IC1.37 (PC6)
- net PC9: now reaches IC1.40 (PC9)
- net LENC2: now reaches IC1.41 (PA8)
- net LENC1: now reaches IC1.42 (PA9)
- net RENC2: now reaches IC1.56 (PB4)
- net RENC1: now reaches IC1.57 (PB5)
- net PB9: now reaches IC1.62 (PB9)
- net PC0: now reaches IC1.8 (PC0)
- net PC1: now reaches IC1.9 (PC1)
- no-connect marks 47 -> 30
Other:
- note added: "Debug Pin Headers"
- moved on the sheet: C25, C70, C71, C72, C76
